File: Fingerprint Lock/Fingerprint lock_1.2.brd (EAGLE design)
At the start: 160 x 100 mm, 14 parts, among them J4 POWER_JACK, U1 NCP1117ST50T3G, U2 FT232RL, U4 ATMEGA328P-PU, X1 CSTCE16M0V53-R0 16MHZ

Commit message: Add files via upload
Parts:
- added J1: 9V, SparkFun-Connectors:BC9VPC
- added R3: 0, rcl:R0805
- added T1: TIP122, transistor:TO220
- moved U1 117.5 mm to (22.9, 63.5)
- moved JP3 100.4 mm to (62.2, 14.0)
- moved D1 94.8 mm to (72.4, 80.0)
- moved C4 86.4 mm to (21.6, 83.8)
- moved C3 70.3 mm to (35.6, 83.8)
- moved J4 64.9 mm to (72.4, 38.1)
- moved C2 60.8 mm to (48.3, 63.5)
- moved X1 51.2 mm to (43.2, 40.6)
- moved R1 50.9 mm to (30.5, 58.4)
- moved R2 45.6 mm to (43.2, 35.6)
- moved C6 41.6 mm to (50.8, 83.8)
- moved U4 40.7 mm to (41.9, 50.8)
- moved U2 38.1 mm to (59.7, 63.5)
- moved JP1 34.3 mm to (38.1, 94.0)
Connections:
- new net 9V: J1.V+, JP3.1
- new net N$2: JP1.2, R3.1
- new net N$6: JP3.2, T1.2
- net GND: now also J1.V-, T1.3; no longer JP3.1
- net LOCK: now also T1.1; no longer JP3.2
- net N$5: now also R3.2; no longer JP1.2
Routing:
- net PWRIN: track 152.9 -> 29.1 mm
- net +5V: track 199.6 -> 122.8 mm
- net GND: track 337.9 -> 282.5 mm, vias 0 -> 1
- net VIN: track 124.1 -> 75.1 mm
- net N$4: track 62.6 -> 32.0 mm
- net N$5: track 55.1 -> 27.2 mm
- net N$2: track 0.00 -> 26.8 mm
- net N$6: track 0.00 -> 23.0 mm
- net N$3: track 57.1 -> 38.0 mm
- net XTAL1: track 30.3 -> 13.0 mm
- net 9V: track 0.00 -> 11.4 mm
- net RESET: track 22.5 -> 13.2 mm
- net XTAL2: track 34.9 -> 26.5 mm
- net LOCK: track 55.9 -> 62.4 mm
- net N$1: track 49.3 -> 54.0 mm
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Other:
- board size 160 x 100 mm -> 90.2 x 100 mm
