File: Fingerprint Lock/Fingerprint lock_1.2.sch (EAGLE design)
At the start: 14 parts, among them J4 POWER_JACK, U1 NCP1117ST50T3G, U2 FT232RL, U4 ATMEGA328P-PU, X1 CSTCE16M0V53-R0 16MHZ

Commit message: Add files via upload
Parts:
- added J1: 9V, SparkFun-Connectors:BC9VPC
- added R3: 0, rcl:R-US_R0805
- added T1: TIP122, transistor:TIP122
Connections:
- new net 9V: J1.V+, JP3.1
- new net N$2: JP1.2, R3.1
- new net N$6: JP3.2, T1.C
- net GND: now also J1.V-, T1.E; no longer JP3.1
- net LOCK: now also T1.B; no longer JP3.2
- net N$5: now also R3.2; no longer JP1.2
Other:
- note added: "9V solenoid"
- note added: "TEST POINT"
Changed lines of the file:
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@@
 <part name="GND1" library="supply1" library_urn="urn:adsk.eagle:library:371" deviceset="GND" device=""/>
 <part name="P+1" library="supply1" library_urn="urn:adsk.eagle:library:371" deviceset="+5V" device=""/>
+<part name="T1" library="transistor" library_urn="urn:adsk.eagle:library:402" deviceset="TIP122" device="" package3d_urn="urn:adsk.eagle:package:28520/1"/>
+<part name="J1" library="SparkFun-Connectors" library_urn="urn:adsk.eagle:library:513" deviceset="BC9VPC" device="" package3d_urn="urn:adsk.eagle:package:38011/1" value="9V"/>
+<part name="U$2" library="Airquality_Sensor" library_urn="urn:adsk.eagle:library:16015176" deviceset="GND" device=""/>
 <part name="U$1" library="Airquality_Sensor" library_urn="urn:adsk.eagle:library:16015176" deviceset="GND" device=""/>
+<part name="R3" library="rcl" library_urn="urn:adsk.eagle:library:334" deviceset="R-US_" device="R0805" package3d_urn="urn:adsk.eagle:package:23553/2" value="0"/>
 </parts>
 <sheets>
@@
 <wire x1="101.6" y1="-2.54" x2="40.64" y2="-2.54" width="0.1524" layer="97"/>
 <text x="55.88" y="-86.36" size="3.81" layer="97">TTL</text>
+<text x="213.36" y="55.88" size="1.778" layer="97">9V solenoid</text>
+<text x="137.16" y="-5.08" size="1.778" layer="97">TEST POINT</text>
 </plain>
 <instances>
@@
 <attribute name="VALUE" x="-22.86" y="59.69" size="1.778" layer="96"/>
 </instance>
-<instance part="GND6" gate="1" x="179.07" y="-2.54" smashed="yes" rot="R270">
-<attribute name="VALUE" x="173.99" y="-5.08" size="1.778" layer="96" rot="R270"/>
+<instance part="GND6" gate="1" x="177.8" y="-6.35" smashed="yes">
+<attribute name="VALUE" x="177.8" y="-8.89" size="1.778" layer="96"/>
 </instance>
 <instance part="JP1" gate="A" x="203.2" y="-2.54" smashed="yes">
@@
 <attribute name="VALUE" x="86.995" y="-7.62" size="1.778" layer="96" rot="R180"/>
 </instance>
-<instance part="U$1" gate="G$1" x="231.14" y="38.1" smashed="yes">
-<attribute name="VALUE" x="229.616" y="35.56" size="1.27" layer="96"/>
+<instance part="T1" gate="G$1" x="203.2" y="76.2" smashed="yes">
+<attribute name="NAME" x="196.85" y="83.82" size="1.778" layer="95"/>
+<attribute name="VALUE" x="199.136" y="81.28" size="1.778" layer="96"/>
+</instance>
+<instance part="J1" gate="G$1" x="238.76" y="53.34" smashed="yes">
+<attribute name="VALUE" x="228.6" y="45.72" size="1.778" layer="96" font="vector"/>
+<attribute name="NAME" x="231.14" y="54.356" size="1.778" layer="95" font="vector"/>
+</instance>
+<instance part="U$2" gate="G$1" x="208.28" y="58.42" smashed="yes">
+<attribute name="VALUE" x="206.756" y="55.88" size="1.27" layer="96"/>
+</instance>
+<instance part="U$1" gate="G$1" x="223.52" y="35.56" smashed="yes">
+<attribute name="VALUE" x="221.996" y="33.02" size="1.27" layer="96"/>
+</instance>
+<instance part="R3" gate="G$1" x="142.24" y="1.27" smashed="yes" rot="R180">
+<attribute name="NAME" x="146.05" y="-0.2286" size="1.778" layer="95" rot="R180"/>
+<attribute name="VALUE" x="146.05" y="4.572" size="1.778" layer="96" rot="R180"/>
 </instance>
 </instances>
@@
 </segment>
 <segment>
-<pinref part="GND6" gate="1" pin="GND"/>
-<pinref part="JP1" gate="A" pin="4"/>
-<wire x1="181.61" y1="-2.54" x2="200.66" y2="-2.54" width="0.1524" layer="91"/>
-</segment>
-<segment>
 <pinref part="U2" gate="G$1" pin="GND1"/>
 <wire x1="73.66" y1="-63.5" x2="86.36" y2="-63.5" width="0.1524" layer="91"/>
@@
 </segment>
 <segment>
-<pinref part="JP3" gate="G$1" pin="1"/>
-<wire x1="220.98" y1="63.5" x2="231.14" y2="63.5" width="0.1524" layer="91"/>
-<wire x1="231.14" y1="63.5" x2="231.14" y2="40.64" width="0.1524" layer="91"/>
+<pinref part="T1" gate="G$1" pin="E"/>
+<wire x1="208.28" y1="68.58" x2="208.28" y2="60.96" width="0.1524" layer="91"/>
+<pinref part="U$2" gate="G$1" pin="GND"/>
+</segment>
+<segment>
+<pinref part="J1" gate="G$1" pin="V-"/>
+<wire x1="238.76" y1="43.18" x2="223.52" y2="43.18" width="0.1524" layer="91"/>
 <pinref part="U$1" gate="G$1" pin="GND"/>
+<wire x1="223.52" y1="43.18" x2="223.52" y2="38.1" width="0.1524" layer="91"/>
+</segment>
+<segment>
+<pinref part="JP1" gate="A" pin="4"/>
+<wire x1="200.66" y1="-2.54" x2="177.8" y2="-2.54" width="0.1524" layer="91"/>
+<pinref part="GND6" gate="1" pin="GND"/>
+<wire x1="177.8" y1="-2.54" x2="177.8" y2="-3.81" width="0.1524" layer="91"/>
 </segment>
 </net>
@@
 <net name="N$5" class="0">
 <segment>
-<pinref part="JP1" gate="A" pin="2"/>
 <wire x1="106.68" y1="-50.8" x2="106.68" y2="2.54" width="0.1524" layer="91"/>
-<wire x1="106.68" y1="2.54" x2="200.66" y2="2.54" width="0.1524" layer="91"/>
 <pinref part="U2" gate="G$1" pin="3V3OUT"/>
 <wire x1="73.66" y1="-50.8" x2="106.68" y2="-50.8" width="0.1524" layer="91"/>
+<pinref part="R3" gate="G$1" pin="2"/>
+<wire x1="106.68" y1="2.54" x2="137.16" y2="2.54" width="0.1524" layer="91"/>
+<wire x1="137.16" y1="2.54" x2="137.16" y2="1.27" width="0.1524" layer="91"/>
 </segment>
 </net>
@@
 <pinref part="U4" gate="G$1" pin="(SCK)PB5"/>
 <wire x1="8.89" y1="-17.78" x2="25.4" y2="-17.78" width="0.1524" layer="91"/>
-<label x="25.4" y="-22.86" size="1.778" layer="95"/>
-</segment>
-<segment>
-<pinref part="JP3" gate="G$1" pin="2"/>
-<wire x1="220.98" y1="66.04" x2="231.14" y2="66.04" width="0.1524" layer="91"/>
-<wire x1="231.14" y1="66.04" x2="231.14" y2="76.2" width="0.1524" layer="91"/>
-<label x="233.68" y="76.2" size="1.778" layer="95"/>
+<wire x1="25.4" y1="-17.78" x2="25.4" y2="10.16" width="0.1524" layer="91"/>
+<wire x1="25.4" y1="10.16" x2="160.02" y2="10.16" width="0.1524" layer="91"/>
+<wire x1="160.02" y1="10.16" x2="160.02" y2="76.2" width="0.1524" layer="91"/>
+<pinref part="T1" gate="G$1" pin="B"/>
+<wire x1="160.02" y1="76.2" x2="200.66" y2="76.2" width="0.1524" layer="91"/>
 </segment>
 </net>
@@
 </segment>
 </net>
+<net name="N$6" class="0">
+<segment>
+<pinref part="T1" gate="G$1" pin="C"/>
+<wire x1="208.28" y1="78.74" x2="238.76" y2="78.74" width="0.1524" layer="91"/>
+<pinref part="JP3" gate="G$1" pin="2"/>
+<wire x1="238.76" y1="78.74" x2="238.76" y2="66.04" width="0.1524" layer="91"/>
+<wire x1="238.76" y1="66.04" x2="220.98" y2="66.04" width="0.1524" layer="91"/>
+</segment>
+</net>
+<net name="9V" class="0">
+<segment>
+<pinref part="JP3" gate="G$1" pin="1"/>
+<wire x1="220.98" y1="63.5" x2="238.76" y2="63.5" width="0.1524" layer="91"/>
+<pinref part="J1" gate="G$1" pin="V+"/>
+<wire x1="238.76" y1="63.5" x2="238.76" y2="60.96" width="0.1524" layer="91"/>
+</segment>
+</net>
+<net name="N$2" class="0">
+<segment>
+<pinref part="R3" gate="G$1" pin="1"/>
+<pinref part="JP1" gate="A" pin="2"/>
+<wire x1="147.32" y1="1.27" x2="200.66" y2="1.27" width="0.1524" layer="91"/>
+<wire x1="200.66" y1="1.27" x2="200.66" y2="2.54" width="0.1524" layer="91"/>
+</segment>
+</net>
